Commit message: fixed the kinect frame name in the urdf and restarted the rviz file w/ new rviz

File: extra/mecanumbot.urdf (robot description, URDF)
Before this commit: robot origins, 4 links, 3 joints
Links:
- removed link openni_camera
- added link camera_link; visual box size=0.06 .28 .03
Joints:
- removed joint base_link_to_openni_camera
- added joint base_link_to_camera_link: type fixed, parent base_link, child camera_link, origin xyz=-0.112 0.0 0.230 rpy=0 -0.05 0
